File: hardware/CH572.kicad_sch (KiCad schematic)
At the start: 15 parts, among them J1 Conn_01x07, J4 USB_C_Receptacle_USB2.0_14P, J5 Conn_01x07, SW1 SW_Push, SW2 SW_Push, U1 CH572D, Y1 32MHz

Commit message: Stash
Parts:
- added D2, D3: LED, LED_SMD:LED_0402_1005Metric, symbol Device:LED
- added R5, R6: 1.5k, Resistor_SMD:R_0402_1005Metric, symbol Device:R
- J1, J5: footprint Connector_PinHeader_2.54mm:PinHeader_1x07_P2.54mm_Vertical -> PCM_ckl-castellated-2.54mm:Castellated_1x07_P2.54mm_Vertical
- R1: LCSC Part # C2933074 -> C25867
- R2, R3, R4: LCSC Part # C105872 -> C2906874
Connections:
- net +3V3: now also R5.2, R6.2
- net PA4: now also D2.1 (K)
- net PA5: now also D3.1 (K)
- new net: D2.2 (A), R5.1
- new net: D3.2 (A), R6.1
